File: lumberjack.kicad_pcb (KiCad board)
At the start: 2 copper layers, 285.4 x 94.9 mm, 156 parts, among them J1 USB, J2 AVR_ISP_6, J3 JST, SW1 RESET, SW2 BOOT, U1 ATMEGA328-PU, Y1 16MHz

Commit message: Delete shit, change footprints to Alps+SI
Parts:
- removed REF**: flags, lumberjack:Flags
- removed REF**: OSHW-Logo_7.5x8mm_Copper, Symbol:OSHW-Logo_7.5x8mm_Copper
- 2u_MX30, 2u_MX60: footprint lumberjack:MX_PCB_200B -> Alps:ALPS-SI-MXStab-2U
- MX1, MX10, MX11, MX12, MX13, MX14, MX15, MX16, MX17, MX18, MX19, MX2, MX20, MX21, MX22, MX23, MX24, MX25, MX26, MX27, MX28, MX29, MX3, MX30, MX31, MX32, MX33, MX34, MX35, MX36, MX37, MX38, MX39, MX4, MX40, MX41, MX42, MX43, MX44, MX45, MX46, MX47, MX48, MX49, MX5, MX50, MX51, MX52, MX53, MX54, MX55, MX56, MX57, MX58, MX59, MX6, MX60, MX7, MX8, MX9: footprint lumberjack:MX -> Alps:ALPS-SI-1U
- turned MX8 to 0 degrees
Routing:
- net Net-(D4-Pad2): track 111.7 -> 211.1 mm
- net /COL0: track 259.9 -> 160.5 mm
Other:
- net class 5v removed
- net class Default removed
- board text removed: "Lumberjack rev1.3 u/peejeh 03/2021"
