File: lumberjerk.kicad_pcb (KiCad board)
At the start: 2 copper layers, 285.4 x 94.9 mm, 135 parts, among them J2 SM04B-SRSS-TB(LF)(SN), J3 SM04B-SRSS-TB(LF)(SN), SW1 SW_Push, U1 ProMicro

Commit message: Finalize design, add gerbers
Parts:
- added H10: logo, silks:falcon, F.Cu at (152.4, 89.6)
Routing:
- net Col1: track 300.6 -> 298.4 mm
- net Col10: track 270.6 -> 268.7 mm
- net Col0: track 317.0 -> 315.3 mm
- net Col2: track 282.8 -> 281.1 mm
- net Col3: track 265.8 -> 264.1 mm
- net Col4: track 248.7 -> 247.0 mm
- net Col11: track 286.3 -> 284.9 mm
- net Col9: track 252.3 -> 250.8 mm
- net Col8: track 235.2 -> 233.8 mm
- net Col7: track 218.2 -> 216.9 mm
- net USBGND: track 162.9 -> 162.3 mm
Other:
- board text added: "Lumberjerk designed by Gvalch'ca with <3 Inspired by the Lumberjack github.com/peej/lumberjack-keyboard"
