File: lumberjerk.kicad_sch (KiCad schematic)
At the start: 135 parts, among them J2 SM04B-SRSS-TB(LF)(SN), J3 SM04B-SRSS-TB(LF)(SN), SW1 SW_Push, U1 ProMicro

Commit message: Finalize design, add gerbers
Parts:
- added H10: logo, silks:falcon, symbol Mechanical:MountingHole
Changed lines of the file:
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@@
     (pin "2")
+  )
+  (symbol (lib_id "Mechanical:MountingHole") (at 167.64 166.37 0) (unit 1)
+    (in_bom yes) (on_board yes)
+    (property "Reference" "H10" (id 0) (at 170.18 165.2016 0)
+      (effects (font (size 1.27 1.27)) (justify left))
+    )
+    (property "Value" "logo" (id 1) (at 170.18 167.513 0)
+      (effects (font (size 1.27 1.27)) (justify left))
+    )
+    (property "Footprint" "silks:falcon" (id 2) (at 167.64 166.37 0)
+      (effects (font (size 1.27 1.27)) hide)
+    )
+    (property "Datasheet" "~" (id 3) (at 167.64 166.37 0)
+      (effects (font (size 1.27 1.27)) hide)
+    )
   )
   (symbol (lib_id "MX_Alps_Hybrid:MX-NoLED") (at 162.56 36.83 90) (mirror x) (unit 1)
@@
       (effects (font (size 1.524 1.524)) hide)
     )
+    (pin "1")
+    (pin "2")
+    (pin "3")
+    (pin "4")
     (pin "5")
-    (pin "4")
-    (pin "3")
-    (pin "2")
-    (pin "1")
   )
   (symbol (lib_id "Device:D_Small") (at 67.31 43.18 90) (unit 1)
@@
       (reference "H9") (unit 1) (value "M2") (footprint "Schematic Library:poker-screw-normal")
     )
+    (path "/274465f0-41e7-4702-aa90-f3037c193441"
+      (reference "H10") (unit 1) (value "logo") (footprint "silks:falcon")
+    )
     (path "/33148e9e-7e70-49cb-92ac-da1cc6128eeb"
